Commit message: Simulation working with position controller

File: Workspace/src/antenna_sim_description/com_base_station/model.urdf (robot description, URDF)
Before this commit: robot com_base_station, 3 links, 2 joints
Joints:
- joint antenna_base_to_antenna: limit effort=30 velocity=1.0 -> effort=30 velocity=0.5
